File: [05] PCB Design/KiCad/Forward_Converter/Forward_Converter.kicad_sch (KiCad schematic)
At the start: 18 parts, among them Q1 CSD19534Q5A, Q2 CSD19534Q5A, Q3 BSC320N20NS3G, Q4 BCX56, T1 P0926NL, U1 LT1952EGN-1-PBF, U2 LTC3900ES8-PBF, U3 MC7812CDTRKG, U4 LT4430ES6-TRPBF

Commit message: Schematic update
IC's are updated, transformer is added
Parts:
- added C10, C6: 10nF, symbol Device:C
- added C11, C12, C13, C9: C, symbol Device:C
- added C14, C15: 1uF, symbol Device:C
- added C16: 2.2nF, symbol Device:C
- added C17: 10pF, symbol Device:C
- added C4, C5: 100nF, symbol Device:C
- added C7: 100pF, symbol Device:C
- added C8: 220pF, symbol Device:C
- added J1, J2: Conn_01x02_Pin, symbol Connector:Conn_01x02_Pin
- added Q5: BC857, Package_TO_SOT_SMD:SOT-23, symbol Transistor_BJT:BC857
- added R1: 1R, symbol Device:R
- added R10: 180k, symbol Device:R
- added R11, R13, R14, R15, R16, R18, R2, R24, R4, R5, R6, R7: 10k, symbol Device:R
- added R12: 100k, symbol Device:R
- added R17, R19: 10k, Resistor_SMD:R_0805_2012Metric, symbol Device:R
- added R20, R8: 47R, symbol Device:R
- added R21, R22: R, symbol Device:R
- added R23: 8.2k, symbol Device:R
- added R25: 1.2k, symbol Device:R
- added R26: 220R, symbol Device:R
- added R27: 22k, symbol Device:R
- added R3: 10m, symbol Device:R
- added R9: 33k, symbol Device:R
- added U5: TCMT1106, Package_SO:SOP-4_4.4x2.6mm_P1.27mm, symbol Isolator:TCMT1106
- T2: value ~ -> EE30157-Custom; footprint (none) -> Forward_Footprint:EE30157-Custom
Connections:
- net GND: now also T1.6, U1.4 (SYNC), U1.8 (GND), C4.1, C5.1, C6.1, C7.1, Q5.3 (C), R10.2, R11.2, R12.2, R2.2, R25.2, R3.2, R5.2, R7.2
- net Vout: now reaches C3.1, L2.2
- net Vout: now also C11.1, C12.1, C13.1, J2.1 (Pin_1), R21.1
- net GNDSEC: now reaches C3.2, Q1.1 (S), Q1.2 (S), Q1.3 (S), Q2.1 (S), Q2.2 (S), Q2.3 (S)
- net GNDSEC: now also T1.3, U2.6 (GND), U4.2 (GND), C10.1, C11.2, C12.2, C13.2, C14.2, C15.2, C9.2, J2.2 (Pin_2), R14.1, R15.1, R17.2, R19.2, R22.2, U5.3
- net Vin: now reaches T2.3
- net Vin: now also T2.5, J1.1 (Pin_1), R6.1
- net at T2.4: now also Q3.5 (D)
- net VSEC: now reaches L1.1, Q2.5 (D), T2.7
- net VSEC: now also R13.1
- net at U1.1 (COMP): now also R9.1
- net at U1.10 (ISENSE): now also U1.11 (OC), C6.2, R8.1
- net at U1.12 (DELAY): now also R12.1
- net PGND: now reaches U1.13 (PGND)
- net PGND: now also J1.2 (Pin_2)
- net GATEOUT: now reaches U1.14 (OUT)
- net GATEOUT: now also R1.2
- net Vcont: now reaches U1.15 (VIN)
- net Vcont: now also R26.1
- net SOUT: now reaches U1.16 (SOUT)
- net SOUT: now also C7.2, C8.2
- net FB: now reaches U1.2 (FB)
- net FB: now also R27.1, R9.2
- net at U1.3 (ROSC): now also R10.1
- net at U1.5 (SS_MAXDC): now also C5.2, R4.1, R7.1
- net VREF: now reaches U1.6 (VREF)
- net VREF: now also C4.2, Q5.1 (B), R4.2
- net at U1.7 (SD_VSEC): now also R5.1, R6.2
- net at U1.9 (BLANK): now also R11.1
- net at U4.1 (VIN): now also C14.1
- net at U4.3 (OC): now also C15.1
- net at U4.4 (FB): now also C16.1, C17.1, R21.2, R22.1
- net at U4.5 (COMP): now also C17.2, R23.1
- net at U4.6 (OPTO): now also R24.2
- net at Q1.4 (G): now also R16.2, R17.1
- net at U2.1 (CS+): now also R13.2, R14.2
- net at U2.2 (CS-): now also R15.2
- net CG: now reaches U2.3 (CG)
- net CG: now also R18.1
- net Vbias: now reaches U2.4 (VCC)
- net Vbias: now also C9.1, R20.2
- net FG: now reaches U2.5 (FG)
- net FG: now also R16.1
- net at U2.7 (TIMER): now also C10.2, R20.1
- net at U2.8 (SYNC): now also T1.4
- net Isense: now reaches Q3.1 (S), Q3.2 (S), Q3.3 (S)
- net Isense: now also R3.1, R8.2
- net at Q3.4 (G): now also R1.1, R2.1
- net at T1.1: now also C8.1
- net at Q2.4 (G): now also R18.2, R19.1
- new net: C16.2, R23.2
- new net: Q5.2 (E), R25.1, R27.2, U5.2
- new net: R26.2, U5.1
- new net: R24.1, U5.4
- no-connect marks 0 -> 2
Other:
- note added: "External Voltage Supply Konnektör Eklenecek"
- moved on the sheet: C1, C2, C3, D1, D2, L1, L2, L3, Q1, Q2, Q3, Q4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

Commit message: Schematic Update
Almost Complete
Parts:
- removed D1, D2: MBR0540, Diode_SMD:D_SOD-123, symbol Diode:MBR0540
- added C18, C19, C20: C, symbol Device:C
- added C21: 1uF, symbol Device:C
- added D1, D2, D3, D4: MS110, Diode_SMD:D_SMA, symbol Diode:MBRA340
- added D10: 1SMA5931, Diode_SMD:D_SMA, symbol Device:D_Zener
- added D5, D9: SMAJ7.5A, Diode_SMD:D_SMA, symbol Diode:SMAJ7.5A
- added D6, D7: D_Schottky, Diode_SMD:D_SMA, symbol Device:D_Schottky
- added D8: BR320, Diode_SMD:D_SMA, symbol Diode:MBRA340
- added L4: 22uH, Inductor_SMD:L_12x12mm_H6mm, symbol Device:L
- added Q6: BCX56, Package_TO_SOT_SMD:SOT-89-3, symbol Transistor_BJT:BCX56
- added R28: 1k, symbol Device:R
- added R29, R30: 4.7k, symbol Device:R
- C2: value C -> 22uF
- L3: value 10uH -> 22uH
Connections:
- net CG: now also D7.1 (K)
- net FG: now also D6.1 (K)
- net GND: now also C18.2, D8.2 (A); no longer C2.2
- net GNDSEC: now also T2.10, U5.2, C20.2, D2.2 (A), D5.2 (A2); no longer U5.3
- net Vbias: now also Q4.3 (E), C19.1, C21.1, D10.1 (K), Q6.3 (E), R30.2
- net Vcont: now also C2.1, L3.1, Q6.2 (C), R29.2
- net Vin: now also T2.1, R30.1; no longer T2.3, T2.5
- net Vaux: now reaches C1.1, U3.3 (VO)
- net at L3.2: now also D1.1 (K), D4.1 (K)
- net Vsw: now reaches T2.2
- net Vsw: now also Q3.5 (D)
- net AUX: now reaches T2.4
- net AUX: now also D4.2 (A); no longer Q3.5 (D)
- net VSEC_GND: now reaches Q1.5 (D), T2.8
- net at Q5.2 (E), R25.1, R27.2: now also U5.3; no longer U5.2
- net at U5.1: now also R24.1; no longer R26.2
- net at U5.4: now also R26.2; no longer R24.1
- net at Q1.4 (G), R16.2, R17.1: now also D6.2 (A)
- net at Q2.4 (G), R18.2, R19.1: now also D7.2 (A)
- net at Q4.1 (B): now also C19.2, D5.1 (A1), R28.1
- net at Q4.2 (C): now also C20.1, L4.1, R28.2
- new net: C2.2, C21.2, D1.2 (A), D10.2 (A), D9.2 (A2), T2.5
- new net: D9.1 (A1), Q6.1 (B), R29.1
- new net: C18.1, U3.1 (VI)
- new net: D2.1 (K), D3.1 (K), L4.2
- new net RST: D8.1 (K), T2.3
Other:
- moved on the sheet: C1, C10, C9, J1, Q4, R13, R14, R15, R20, R24, U2, U3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
